File: pd-adapter/pd-adapter.kicad_pcb (KiCad board)
At the start: 4 copper layers, 45 x 38 mm, 59 parts, among them J1 USB, J2 DBG, J3 EXT, SW1 RST, SW2 USER, U1 FUSB302BMPX, U2 TPS54202DDC, U3 STM32F072C8Tx

Commit message: First pass at adapter layout, needs second revision
Connections:
- U3 pad 13: /EXT_3 -> Net-(U3-Pad13)
- U3 pad 14: /EXT_4 -> Net-(U3-Pad14)
- U3 pad 25: Net-(U3-Pad25) -> /EXT_4
- U3 pad 26: Net-(U3-Pad26) -> /EXT_3
Routing:
- net +3V3: track 22.1 -> 58.0 mm, vias 0 -> 14
- net VBUS: track 7.80 -> 40.5 mm, vias 0 -> 3
- net /SWDIO: track 0.00 -> 29.8 mm, vias 0 -> 1
- net /LED_GRN: track 0.00 -> 27.1 mm, vias 0 -> 2
- net /D-: track 30.4 -> 54.1 mm, vias 2 -> 3
- net /LED_RED: track 0.00 -> 23.5 mm, vias 0 -> 2
- net /SDA_EXT: track 0.00 -> 22.9 mm, vias 0 -> 2
- net /~RST: track 14.4 -> 36.9 mm, vias 3 -> 4
- net /D+: track 32.4 -> 53.2 mm, vias 2 -> 3
- net /LED_YLL: track 0.00 -> 20.2 mm, vias 0 -> 2
- net /SWCLK: track 0.00 -> 20.1 mm, vias 0 -> 1
- net /SWO: track 0.00 -> 18.0 mm, vias 0 -> 3
- net /EXT_4: track 0.00 -> 17.1 mm, vias 0 -> 1
- net /EXT_3: track 0.00 -> 15.5 mm, vias 0 -> 1
- net /SBU1: track 32.3 -> 47.4 mm, vias 2 -> 4
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- added copper zone on In2.Cu, net +3V3
- added copper zone on In1.Cu, net VBUS

Commit message: Finished it, one more pair of eyes and it can go into production
Parts:
- added J3: EXT, Connector_PinHeader_2.54mm:PinHeader_1x06_P2.54mm_Vertical, F.Cu at (163.0, 95.5)
- added J5: EXT, Connector_PinHeader_2.54mm:PinHeader_1x04_P2.54mm_Vertical, F.Cu at (163.0, 120.9)
- added R7: 4.7k, Resistor_SMD:R_0603_1608Metric, F.Cu at (157.2, 115.1)
- added R9: 4.7k, Resistor_SMD:R_0603_1608Metric, F.Cu at (157.2, 112.0)
- H5: value MountingHole -> Transistor
- H6: value MountingHole -> Logo; footprint Automated:fully_automated_logo_soldermask -> Automated:fully_automated_logo_silkscreen
- J4: renamed from J3; value EXT -> Qwiic; footprint Connector_PinHeader_2.54mm:PinHeader_1x12_P2.54mm_Vertical -> Connector_JST:JST_SH_SM04B-SRSS-TB_1x04-1MP_P1.00mm_Horizontal
- moved TP2 35.8 mm to (122.1, 103.5)
- moved TP1 35.8 mm to (125.4, 103.5)
- moved J4 16.6 mm to (161.4, 114.6), turned to 90 degrees
- moved R8 13.6 mm to (149.8, 118.7), turned to 270 degrees
- moved R1 13.6 mm to (140.8, 108.7), turned to 270 degrees
- moved R2 13.6 mm to (139.2, 108.7), turned to 270 degrees
- moved C12 13.0 mm to (154.2, 116.8), turned to 270 degrees
- moved C15 9.38 mm to (144.2, 116.0), turned to 180 degrees
- moved C9 2.64 mm to (141.9, 118.1)
- moved C11 2.60 mm to (147.2, 106.0), turned to 0 degrees
- moved C14 1.66 mm to (142.8, 114.4), turned to 0 degrees
- moved C1 1.41 mm to (133.1, 99.9)
- moved C2 1.41 mm to (130.0, 102.3)
- moved C5 1.41 mm to (135.8, 103.1)
- moved C6 1.41 mm to (139.7, 102.4)
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- renumbered R8 to R10, R9 to R11, R10 to R12, R11 to R13, R12 to R14, R13 to R15, R7 to R8
Connections:
- J4 pad 1: VBUS -> GND
- J4 pad 3: GND -> /SDA_EXT
- J4 pad 4: /SCK -> /SCL_EXT
- U3 pad 12: /EXT_2 -> /SBU1
- U3 pad 13: Net-(U3-Pad13) -> /SBU2
- U3 pad 16: /MIPO -> /CIPO
- U3 pad 17: /MOPI -> /COPI
- U3 pad 18: /LED_YLL -> /LED_WHT
- U3 pad 19: Net-(U3-Pad19) -> /LED_YLL
- U3 pad 2: /~INT -> /EXT_4
- U3 pad 21: /SCL -> Net-(U3-Pad21)
- U3 pad 22: /SDA -> /LED_BLU
- U3 pad 25: /EXT_4 -> Net-(U3-Pad25)
- U3 pad 26: /EXT_3 -> /SCL
- U3 pad 27: /LED_WHT -> /SDA
- U3 pad 28: /LED_BLU -> /~INT
- U3 pad 29: /EXT_1 -> Net-(U3-Pad29)
- U3 pad 3: Net-(U3-Pad3) -> /EXT_3
- U3 pad 4: Net-(U3-Pad4) -> /EXT_2
- U3 pad 42: /SBU1 -> Net-(U3-Pad42)
- U3 pad 43: /SBU2 -> Net-(U3-Pad43)
- U3 pad 5: Net-(U3-Pad5) -> /EXT_1
Routing:
- net /MIPO: track 18.8 -> 0.00 mm, vias 1 -> 0
- net /MOPI: track 17.0 -> 0.00 mm, vias 2 -> 0
- net /SWCLK: track 20.1 -> 37.0 mm, vias 1 -> 2
- net /COPI: track 0.00 -> 15.0 mm
- net /LED_GRN: track 27.1 -> 12.4 mm, vias 2 -> 0
- net /~RST: track 36.9 -> 51.2 mm, vias 4 -> 5
- net /CIPO: track 0.00 -> 13.5 mm
- net GND: track 60.3 -> 48.0 mm, vias 18 -> 17
- net /SWO: track 18.0 -> 30.1 mm, vias 3 -> 2
- net /SDA_EXT: track 22.9 -> 11.4 mm
- net /LED_RED: track 23.5 -> 13.2 mm, vias 2 -> 0
- net /SCL: track 26.9 -> 36.7 mm, vias 1 -> 2
- net /SCK: track 22.6 -> 13.0 mm, vias 3 -> 0
- net /LED_BLU: track 31.5 -> 23.4 mm, vias 0 -> 4
- net /SCL_EXT: track 19.7 -> 12.3 mm, vias 1 -> 2
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- added copper zone on F.Cu, net VBUS
- removed copper zone on In1.Cu, net VBUS
Other:
- board text added: "CIPÓ"
- board text added: "COPI"
- board text added: "June 2020, v0.1"
- board text added: "automated.ee"
- board text removed: "MIPO"
- board text removed: "MOPI"
- board text removed: "SCL"
- board text removed: "SDA"
