File: pd-adapter/pd-adapter.sch (KiCad schematic (older format))
At the start: 41 parts

Commit message: LED stonks
Parts:
- removed C? (x2): 100nF, Capacitor_SMD:C_0603_1608Metric, symbol Device:C_Small
- removed C? (x5): 100nF/50V, Capacitor_SMD:C_0603_1608Metric, symbol Device:C_Small
- removed R? (x3): 4.7k, Resistor_SMD:R_0603_1608Metric, symbol Device:R_Small
- added C? (x2): 100nF, Capacitor_SMD:C_0603_1608Metric, symbol Device:C_Small
- added C? (x5): 100nF/50V, Capacitor_SMD:C_0603_1608Metric, symbol Device:C_Small
- added D?: Red/2V, LED_SMD:LED_0603_1608Metric_Castellated, symbol Device:LED_Small
- added D?: White/2.9V, LED_SMD:LED_0603_1608Metric_Castellated, symbol Device:LED_Small
- added D?: Blue/2.8V, LED_SMD:LED_0603_1608Metric_Castellated, symbol Device:LED_Small
- added D?: Green/3.3V, LED_SMD:LED_0603_1608Metric_Castellated, symbol Device:LED_Small
- added D?: Yellow/2.9V, LED_SMD:LED_0603_1608Metric_Castellated, symbol Device:LED_Small
- added R? (x3): 4.7k, Resistor_SMD:R_0603_1608Metric, symbol Device:R_Small
- added R? (x2): 130, Resistor_SMD:R_0603_1608Metric, symbol Device:R_Small
- added R? (x2): 47, Resistor_SMD:R_0603_1608Metric, symbol Device:R_Small
- added R?: 0, Resistor_SMD:R_0603_1608Metric, symbol Device:R_Small
- added TP?: SDA, TestPoint:TestPoint_THTPad_D2.5mm_Drill1.2mm, symbol Connector:TestPoint_Small
- added TP?: SCL, TestPoint:TestPoint_THTPad_D2.5mm_Drill1.2mm, symbol Connector:TestPoint_Small
- added TP?: SBU1, TestPoint:TestPoint_THTPad_D2.5mm_Drill1.2mm, symbol Connector:TestPoint_Small
- added TP?: SBU2, TestPoint:TestPoint_THTPad_D2.5mm_Drill1.2mm, symbol Connector:TestPoint_Small
- C?: value 1uF/50V -> 10uF/10V; MPN CL10A105KB8NNNC -> CL10A106KP8NNNC
- J? (x2): MPN (none) -> DNP
- SW?: footprint (none) -> Automated:SW_SPST_PTS636_G; MPN (none) -> DNP
Connections:
- net +3V3: now also C?.1, C?.1, C?.1, C?.1, C?.1, C?.1, R?.1, R?.1, R?.1, R?.1, R?.1, R?.1, R?.1, R?.1
- net GND: now also C?.2, C?.2, C?.2, C?.2, C?.2, C?.2, C?.2
- net SBU1: now also TP?.1
- net SBU2: now also TP?.1
- net SCL: now also R?.2, TP?.1
- net SDA: now also R?.2, TP?.1
- net ~INT: now also R?.2
- net ~RST: now also C?.1
- net LED_YLL: now reaches U?.18 (PB0)
- net LED_YLL: now also D?.1 (K)
- net LED_WHT: now reaches U?.27 (PB14)
- net LED_WHT: now also D?.1 (K)
- net LED_BLU: now reaches U?.28 (PB15)
- net LED_BLU: now also D?.1 (K)
- net LED_RED: now reaches U?.40 (PB4)
- net LED_RED: now also D?.1 (K)
- net LED_GRN: now reaches U?.41 (PB5)
- net LED_GRN: now also D?.1 (K)
- new net: D?.2 (A), R?.2 (x5)
- no-connect marks 15 -> 10
Other:
- note added: "5x"
- moved on the sheet: R?, SW?, U?

Commit message: Mounting holes and logos
Parts:
- added H? (x4): MountingHole, MountingHole:MountingHole_3.2mm_M3_ISO14580_Pad, symbol Mechanical:MountingHole
Changed lines of the file:
@@
 Wire Wire Line
 	5500 3400 5950 3400
+$Comp
+L Mechanical:MountingHole H?
+U 1 1 5F2310D7
+P 5400 7100
+F 0 "H?" H 5500 7100 50  0000 L CNN
+F 1 "MountingHole" H 5500 7055 50  0001 L CNN
+F 2 "MountingHole:MountingHole_3.2mm_M3_ISO14580_Pad" H 5400 7100 50  0001 C CNN
+F 3 "~" H 5400 7100 50  0001 C CNN
+	1    5400 7100
+	1    0    0    -1
+$EndComp
+$Comp
+L Mechanical:MountingHole H?
+U 1 1 5F231718
+P 5700 7100
+F 0 "H?" H 5800 7100 50  0000 L CNN
+F 1 "MountingHole" H 5800 7055 50  0001 L CNN
+F 2 "MountingHole:MountingHole_3.2mm_M3_ISO14580_Pad" H 5700 7100 50  0001 C CNN
+F 3 "~" H 5700 7100 50  0001 C CNN
+	1    5700 7100
+	1    0    0    -1
+$EndComp
+$Comp
+L Mechanical:MountingHole H?
+U 1 1 5F23192A
+P 5700 7300
+F 0 "H?" H 5800 7300 50  0000 L CNN
+F 1 "MountingHole" H 5800 7255 50  0001 L CNN
+F 2 "MountingHole:MountingHole_3.2mm_M3_ISO14580_Pad" H 5700 7300 50  0001 C CNN
+F 3 "~" H 5700 7300 50  0001 C CNN
+	1    5700 7300
+	1    0    0    -1
+$EndComp
+$Comp
+L Mechanical:MountingHole H?
+U 1 1 5F231B9E
+P 5400 7300
+F 0 "H?" H 5500 7300 50  0000 L CNN
+F 1 "MountingHole" H 5500 7255 50  0001 L CNN
+F 2 "MountingHole:MountingHole_3.2mm_M3_ISO14580_Pad" H 5400 7300 50  0001 C CNN
+F 3 "~" H 5400 7300 50  0001 C CNN
+	1    5400 7300
+	1    0    0    -1
+$EndComp
+$Comp
+L Graphic:SYM_Arrow45_Normal #SYM?
+U 1 1 5F2328C0
+P 6100 7100
+F 0 "#SYM?" H 6250 7150 50  0001 C CNN
+F 1 "SYM_Arrow45_Normal" H 6100 7000 50  0001 C CNN
+F 2 "Automated:transistor_10x10mm" H 6100 7100 50  0001 C CNN
+F 3 "~" H 6100 7100 50  0001 C CNN
+	1    6100 7100
+	1    0    0    -1
+$EndComp
+$Comp
+L Graphic:SYM_Arrow45_Normal #SYM?
+U 1 1 5F232EDA
+P 6100 7300
+F 0 "#SYM?" H 6250 7350 50  0001 C CNN
+F 1 "SYM_Arrow45_Normal" H 6100 7200 50  0001 C CNN
+F 2 "Automated:fully_automated_logo_silkscreen" H 6100 7300 50  0001 C CNN
+F 3 "~" H 6100 7300 50  0001 C CNN
+	1    6100 7300
+	1    0    0    -1
+$EndComp
 $EndSCHEMATC

Commit message: Progress
Parts:
- removed C? (x2): 12pF, Capacitor_SMD:C_0402_1005Metric, symbol Device:C_Small
- removed R?: 390, Resistor_SMD:R_0603_1608Metric, symbol Device:R_Small
- removed Y?: 12MHz, Crystal:Crystal_SMD_3225-4Pin_3.2x2.5mm, symbol Device:Crystal_Small
- added H5: MountingHole, Automated:transistor_10x10mm, symbol Mechanical:MountingHole
- added H6: MountingHole, Automated:fully_automated_logo_soldermask, symbol Mechanical:MountingHole
- added R8: 4.7k, Resistor_SMD:R_0603_1608Metric, symbol Device:R_Small
- added SW2: USER, Automated:SW_SPST_PTS636_G, symbol Switch:SW_Push
- TP1, TP2, TP3, TP4: renamed from TP?; footprint TestPoint:TestPoint_THTPad_D2.5mm_Drill1.2mm -> TestPoint:TestPoint_THTPad_D2.0mm_Drill1.0mm
- gave numbers to parts that had none: 51
Connections:
- net +3V3: now also R8.1
- net EXT_3: now also U3.25 (PB12); no longer U3.13 (PA3)
- net EXT_4: now also U3.26 (PB13); no longer U3.14 (PA4)
- net at U3.10 (PA0): now also SW2.2
- net OSC_IN: no longer names the net of U3.5 (PF0)
- net OSC_OUT: no longer names the net of U3.6 (PF1)
- new net: R8.2, SW2.1
- no-connect marks 10 -> 11

Commit message: First pass at adapter layout, needs second revision
Connections:
- net EXT_3: now also U3.26 (PB13); no longer U3.25 (PB12)
- net EXT_4: now also U3.25 (PB12); no longer U3.26 (PB13)
Changed lines of the file:
@@
 Text Label 10300 2000 0    50   ~ 0
 EXT_1
-Text Label 5600 4000 0    50   ~ 0
+Text Label 5600 4100 0    50   ~ 0
 EXT_3
 Text Label 7550 3000 2    50   ~ 0
@@
 	7550 3000 7250 3000
 Wire Wire Line
-	5950 4000 5600 4000
+	5950 4100 5600 4100
 Text Label 10300 2100 0    50   ~ 0
 EXT_2
@@
 Wire Wire Line
 	10150 1400 10550 1400
-Text Label 5600 4100 0    50   ~ 0
+Text Label 5600 4000 0    50   ~ 0
 EXT_4
 Wire Wire Line
-	5950 4100 5600 4100
+	5950 4000 5600 4000
 Text Label 10300 2300 0    50   ~ 0
 EXT_4

Commit message: Finished it, one more pair of eyes and it can go into production
Parts:
- removed J3: EXT, Connector_PinHeader_2.54mm:PinHeader_1x12_P2.54mm_Vertical, symbol Connector_Generic:Conn_01x12
- added J3: EXT, Connector_PinHeader_2.54mm:PinHeader_1x06_P2.54mm_Vertical, symbol Connector_Generic:Conn_01x06
- added J4: Qwiic, Connector_JST:JST_SH_SM04B-SRSS-TB_1x04-1MP_P1.00mm_Horizontal, symbol Connector_Generic:Conn_01x04
- added J5: EXT, Connector_PinHeader_2.54mm:PinHeader_1x04_P2.54mm_Vertical, symbol Connector_Generic:Conn_01x04
- added R7, R9: 4.7k, Resistor_SMD:R_0603_1608Metric, symbol Device:R_Small
- C1, C10, C11, C12, C13, C14, C3, C5, C9: JLC (none) -> 0603; LCSC (none) -> C14663
- C15, C4, C6, C7: JLC (none) -> 0603; LCSC (none) -> C19702
- C2: JLC (none) -> 1206; LCSC (none) -> C13585
- C8: JLC (none) -> 0603; LCSC (none) -> C39148
- D1, D2, D6, D7: JLC (none) -> SOD-523; LCSC (none) -> C266462
- D10: JLC (none) -> LED_0603; LCSC (none) -> C72043
- D11: JLC (none) -> LED_0603; LCSC (none) -> C2290
- D12: JLC (none) -> LED_0603; LCSC (none) -> C72038
- D3, D4: JLC (none) -> SOD-523; LCSC (none) -> C136161
- D5: JLC (none) -> SOD-323; LCSC (none) -> C22619
- D8: JLC (none) -> LED_0603; LCSC (none) -> C2286; MPN (none) -> KT-0603R
- D9: JLC (none) -> LED_0603; LCSC (none) -> C72041
- H5: value MountingHole -> Transistor
- H6: value MountingHole -> Logo; footprint Automated:fully_automated_logo_soldermask -> Automated:fully_automated_logo_silkscreen
- J1: MPN DNP -> C167321
- L1: JLC (none) -> 1210; LCSC (none) -> C86069
- R1, R2, R3: JLC (none) -> 0603; LCSC (none) -> C23162
- R10: renamed from R8; JLC (none) -> 0603; LCSC (none) -> C23162
- R11: renamed from R9; JLC (none) -> 0603; LCSC (none) -> C23185
- R12: renamed from R10; JLC (none) -> 0603; LCSC (none) -> C23182
- R13: renamed from R11; value 0 -> 10; JLC (none) -> 0603; LCSC (none) -> C22859; MPN 0603WAF0000T5E -> 0603WAF100JT5E
- R14: renamed from R12; JLC (none) -> 0603; LCSC (none) -> C23182
- R15: renamed from R13; JLC (none) -> 0603; LCSC (none) -> C23185
- R4: JLC (none) -> 0603; LCSC (none) -> C23185
- R5: JLC (none) -> 0603; LCSC (none) -> C25803
- R6: JLC (none) -> 0603; LCSC (none) -> C31850
- R8: renamed from R7; JLC (none) -> 0603; LCSC (none) -> C25804
- U1: JLC (none) -> MLP-14_EP_2.5x2.5x0.5P; LCSC (none) -> C132291
- U2: JLC (none) -> SOT-23-6L; LCSC (none) -> C191884
- U3: JLC (none) -> LQFP-48_7.0x7.0x0.5P; LCSC (none) -> C80488
Connections:
- net +3V3: now also J3.2 (Pin_2), J4.2 (Pin_2), R7.1, R9.1
- net EXT_1: now also U3.5 (PF0), J5.1 (Pin_1); no longer U3.29 (PA8)
- net EXT_2: now also U3.4 (PC15), J5.2 (Pin_2); no longer U3.12 (PA2)
- net EXT_3: now also U3.3 (PC14), J5.3 (Pin_3); no longer U3.26 (PB13)
- net EXT_4: now also U3.2 (PC13), J5.4 (Pin_4); no longer U3.25 (PB12)
- net GND: now also J3.3 (Pin_3), J4.1 (Pin_1)
- net LED_BLU: now also U3.22 (PB11); no longer U3.28 (PB15)
- net LED_WHT: now also U3.18 (PB0); no longer U3.27 (PB14)
- net LED_YLL: now also U3.19 (PB1); no longer U3.18 (PB0)
- net SBU1: now also U3.12 (PA2); no longer U3.42 (PB6)
- net SBU2: now also U3.13 (PA3); no longer U3.43 (PB7)
- net SCK: now also J3.6 (Pin_6)
- net SCL: now also U3.26 (PB13); no longer U3.21 (PB10)
- net SCL_EXT: now also J4.4 (Pin_4), R9.2
- net SDA: now also U3.27 (PB14); no longer U3.22 (PB11)
- net SDA_EXT: now also J4.3 (Pin_3), R7.2
- net VBUS: now also J3.1 (Pin_1)
- net ~INT: now also U3.28 (PB15); no longer U3.2 (PC13)
- net MIPO renamed CIPO
- net CIPO: now also J3.5 (Pin_5)
- net MOPI renamed COPI
- net COPI: now also J3.4 (Pin_4)
Other:
- moved on the sheet: J2, TP3, TP4
