File: MCU.sch (KiCad schematic (older format))
At the start: 30 parts

Commit message: almost done
Parts:
- removed D?: B1, symbol Device:LED_Small
- removed D?: P1, symbol Device:LED_Small
- added C?: 100nF, Capacitor_SMD:C_0603_1608Metric, symbol Device:C_Small
- added D? (x2): D_TVS, symbol Device:D_TVS
- added D?: P2, LED_SMD:LED_0603_1608Metric_Castellated, symbol Device:LED_Small
- added D?: B2, LED_SMD:LED_0603_1608Metric_Castellated, symbol Device:LED_Small
- added J?: RS485, symbol Connector_Generic:Conn_01x04
- added J?: EXT, symbol Connector_Generic:Conn_01x04
- added R? (x2): 10k, Resistor_SMD:R_0603_1608Metric, symbol Device:R_Small
- added R?: 100, Resistor_SMD:R_0603_1608Metric, symbol Device:R_Small
- added U?: SP3485CN, Package_SO:SOIC-8_3.9x4.9mm_P1.27mm, symbol Interface_UART:SP3485CN
- D?: footprint (none) -> LED_SMD:LED_0603_1608Metric_Castellated; MPN (none) -> OSB60603C1E
- D?: footprint (none) -> LED_SMD:LED_0603_1608Metric_Castellated; MPN (none) -> OSK40603C1E
- D?: footprint (none) -> LED_SMD:LED_0603_1608Metric_Castellated; MPN (none) -> OSW50603C1E
- J?: footprint (none) -> Connector_USB:USB_C_Receptacle_HRO_TYPE-C-31-M-12
- R? (x5): value 120 -> 100
Connections:
- net +3V3: now also C?.2, R?.1, U?.8 (VCC)
- net Blue2: now also D?.1 (K)
- net D+: now also J?.A6 (D+), J?.B6 (D+), D?.1 (A1)
- net D-: now also J?.A7 (D-), J?.B7 (D-), D?.1 (A1)
- net GND: now also C?.1, D?.2 (A2), D?.2 (A2), R?.2, U?.5 (GND)
- net Pink2: now also D?.1 (K)
- net UART_RX: now also U?.1 (RO)
- net UART_TX: now also U?.4 (DI)
- net EXT1: now reaches U?.15 (PA5)
- net EXT1: now also J?.1 (Pin_1)
- net EXT2: now reaches U?.16 (PA6)
- net EXT2: now also J?.2 (Pin_2)
- net EXT3: now reaches U?.17 (PA7)
- net EXT3: now also J?.3 (Pin_3)
- net ~RE: now reaches U?.25 (PB12)
- net ~RE: now also U?.2 (~RE~)
- net DE: now reaches U?.26 (PB13)
- net DE: now also U?.3 (DE)
- net EXT4: now reaches U?.29 (PA8)
- net EXT4: now also J?.4 (Pin_4)
- net at R?.2: now also D?.2 (A) (x2)
- net ~INT_BQ renamed ~INT_CHG
- new net: J?.1 (Pin_1), J?.3 (Pin_3), R?.1, R?.2, U?.6 (A)
- new net: J?.2 (Pin_2), J?.4 (Pin_4), R?.1, R?.2, U?.7 (B)
- no-connect marks 15 -> 16
Other:
- note added: "TODO: BOOT0 selector switch"
- note removed: "TODO: ESD"
- moved on the sheet: C?, D?, J?, R?, SW?, U?

Commit message: Looks good, just needs some more checking
Parts:
- added J11: CHG, Connector_PinHeader_2.54mm:PinHeader_1x04_P2.54mm_Vertical, symbol Connector_Generic:Conn_01x04
- added TP8: SCL, TestPoint:TestPoint_THTPad_D2.0mm_Drill1.0mm, symbol Connector:TestPoint_Small
- added TP9: SDA, TestPoint:TestPoint_THTPad_D2.0mm_Drill1.0mm, symbol Connector:TestPoint_Small
- J10, J13: renamed from J?; footprint (none) -> Connector_PinHeader_2.54mm:PinHeader_1x04_P2.54mm_Vertical
- J14: renamed from J?; footprint (none) -> Connector_PinHeader_2.54mm:PinHeader_1x02_P2.54mm_Vertical
- gave numbers to parts that had none: 36
Connections:
- net EN_SNK: now also J11.2 (Pin_2)
- net SCL: now also TP8.1
- net SDA: now also TP9.1
- net ~CE: now also J11.1 (Pin_1)
- net ~INT_CHG: now also J11.3 (Pin_3)
- net ~INT_PMC: now also J11.4 (Pin_4)
- net A: now reaches J10.1 (Pin_1), J10.3 (Pin_3), R14.1, R15.2, U5.6 (A)
- net B: now reaches J10.2 (Pin_2), J10.4 (Pin_4), R14.2, R16.1, U5.7 (B)

Commit message: Add some footprints to parts
Parts:
- J9: footprint Connector_USB:USB_C_Receptacle_HRO_TYPE-C-31-M-12 -> Connector_USB:USB_C_Receptacle_XKB_U262-16XN-4BVC11
Changed lines of the file:
@@
 F 0 "J9" H 970 2039 50  0000 R CNN
 F 1 "CTRL" H 970 1948 50  0000 R CNN
-F 2 "Connector_USB:USB_C_Receptacle_HRO_TYPE-C-31-M-12" H 1550 2100 50  0001 C CNN
+F 2 "Connector_USB:USB_C_Receptacle_XKB_U262-16XN-4BVC11" H 1550 2100 50  0001 C CNN
 F 3 "https://www.usb.org/sites/default/files/documents/usb_type-c.zip" H 1550 2100 50  0001 C CNN
 	1    1400 2100

Commit message: Re-annotated, add more footprints
Parts:
- D15: renamed from D14; footprint (none) -> Diode_SMD:D_SOD-123
- D7: renamed from D6; footprint (none) -> Diode_SMD:D_SOD-123
- renumbered D9 to D10, D10 to D11, D11 to D12, D12 to D13, D13 to D14, D5 to D6, D7 to D8, D8 to D9, J9 to J10, J10 to J11, J11 to J12, J12 to J13, J13 to J14, J14 to J15, R14 to R16, R15 to R17, R16 to R18, R17 to R19, R18 to R20, R19 to R21, R20 to R22, R21 to R23, R22 to R24, R23 to R25, R24 to R26, R25 to R27, TP8 to TP7, TP9 to TP8

Commit message: Some more work
Parts:
- SW1, SW2: footprint (none) -> Automated:SW_SPST_PTS636_G; symbol Switch:SW_SPST -> Switch:SW_Push
Changed lines of the file:
@@
 	6200 4250 7800 4250
 $Comp
-L Switch:SW_SPST SW2
+L Switch:SW_Push SW2
 U 1 1 5F0BE69D
 P 4550 3450
-F 0 "SW2" H 4550 3685 50  0000 C CNN
-F 1 "USER" H 4550 3594 50  0000 C CNN
-F 2 "" H 4550 3450 50  0001 C CNN
+F 0 "SW2" H 4550 3735 50  0000 C CNN
+F 1 "USER" H 4550 3644 50  0000 C CNN
+F 2 "Automated:SW_SPST_PTS636_G" H 4550 3450 50  0001 C CNN
 F 3 "~" H 4550 3450 50  0001 C CNN
 	1    4550 3450
@@
 	4300 3450 4350 3450
 $Comp
-L Switch:SW_SPST SW1
+L Switch:SW_Push SW1
 U 1 1 5F0C7422
 P 4200 2750
-F 0 "SW1" H 4200 2985 50  0000 C CNN
-F 1 "RESET" H 4200 2894 50  0000 C CNN
-F 2 "" H 4200 2750 50  0001 C CNN
+F 0 "SW1" H 4200 3035 50  0000 C CNN
+F 1 "RESET" H 4200 2944 50  0000 C CNN
+F 2 "Automated:SW_SPST_PTS636_G" H 4200 2750 50  0001 C CNN
 F 3 "~" H 4200 2750 50  0001 C CNN
 	1    4200 2750
