File: input.sch (KiCad schematic (older format))
At the start: 34 parts

Commit message: I'm pretty happy with it now, will place tomorrow
Connections:
- net labels added: EN_SINK
- net labels removed: EN_SNK
- wire segments 156 -> 157
Other:
- note added: "In a dead battery situation\nwhen EN_SINK goes high,\nACDRV1 should be enabled."
- note removed: "In a dead battery situation\nwhen EN_SNK goes high,\nACDRV1 should be enabled."
- moved on the sheet: R?
Changed lines of the file:
@@
 Connection ~ 4700 1950
 Text Notes 7250 3250 0    50   ~ 0
-In a dead battery situation\nwhen EN_SNK goes high,\nACDRV1 should be enabled.
-Wire Wire Line
-	7850 3450 8300 3450
-Text Label 7850 3450 0    50   ~ 0
-EN_SNK
+In a dead battery situation\nwhen EN_SINK goes high,\nACDRV1 should be enabled.
 $Comp
 L Interface_USB:FUSB307BMPX U?
@@
 L Device:R_Small R?
 U 1 1 5F02F000
-P 10400 3700
-F 0 "R?" H 10341 3654 50  0000 R CNN
-F 1 "10k" H 10341 3745 50  0000 R CNN
-F 2 "Resistor_SMD:R_0603_1608Metric" H 10400 3700 50  0001 C CNN
-F 3 "~" H 10400 3700 50  0001 C CNN
-F 4 "DNP" H 10400 3700 50  0001 C CNN "MPN"
-	1    10400 3700
+P 10650 3700
+F 0 "R?" H 10591 3654 50  0000 R CNN
+F 1 "10k" H 10591 3745 50  0000 R CNN
+F 2 "Resistor_SMD:R_0603_1608Metric" H 10650 3700 50  0001 C CNN
+F 3 "~" H 10650 3700 50  0001 C CNN
+F 4 "DNP" H 10650 3700 50  0001 C CNN "MPN"
+	1    10650 3700
 	-1   0    0    1
 $EndComp
 Wire Wire Line
-	9700 3550 10400 3550
-Wire Wire Line
-	10400 3550 10400 3600
-Connection ~ 10400 3550
+	9700 3550 10650 3550
+Wire Wire Line
+	10650 3550 10650 3600
+Connection ~ 10650 3550
 $Comp
 L power:GND #PWR?
 U 1 1 5F02F009
-P 10400 3900
-F 0 "#PWR?" H 10400 3650 50  0001 C CNN
-F 1 "GND" H 10405 3727 50  0000 C CNN
-F 2 "" H 10400 3900 50  0001 C CNN
-F 3 "" H 10400 3900 50  0001 C CNN
-	1    10400 3900
-	1    0    0    -1
-$EndComp
-Wire Wire Line
-	10400 3900 10400 3800
+P 10650 3900
+F 0 "#PWR?" H 10650 3650 50  0001 C CNN
+F 1 "GND" H 10655 3727 50  0000 C CNN
+F 2 "" H 10650 3900 50  0001 C CNN
+F 3 "" H 10650 3900 50  0001 C CNN
+	1    10650 3900
+	1    0    0    -1
+$EndComp
+Wire Wire Line
+	10650 3900 10650 3800
 Wire Wire Line
 	10150 3150 10150 3200
@@
 L power:+3V3 #PWR?
 U 1 1 5F02F011
-P 10400 3050
-F 0 "#PWR?" H 10400 2900 50  0001 C CNN
-F 1 "+3V3" H 10415 3223 50  0000 C CNN
-F 2 "" H 10400 3050 50  0001 C CNN
-F 3 "" H 10400 3050 50  0001 C CNN
-	1    10400 3050
+P 10650 3050
+F 0 "#PWR?" H 10650 2900 50  0001 C CNN
+F 1 "+3V3" H 10665 3223 50  0000 C CNN
+F 2 "" H 10650 3050 50  0001 C CNN
+F 3 "" H 10650 3050 50  0001 C CNN
+	1    10650 3050
 	1    0    0    -1
 $EndComp
@@
 	10150 3400 10150 3450
 Wire Wire Line
-	10400 3150 10150 3150
-Connection ~ 10400 3150
-Wire Wire Line
-	10400 3150 10400 3300
-Wire Wire Line
-	10400 3500 10400 3550
+	10650 3150 10150 3150
+Connection ~ 10650 3150
+Wire Wire Line
+	10650 3150 10650 3300
+Wire Wire Line
+	10650 3500 10650 3550
 $Comp
 L Device:R_Small R?
 U 1 1 5F02F024
-P 10400 3400
-F 0 "R?" H 10341 3354 50  0000 R CNN
-F 1 "10k" H 10341 3445 50  0000 R CNN
-F 2 "Resistor_SMD:R_0603_1608Metric" H 10400 3400 50  0001 C CNN
-F 3 "~" H 10400 3400 50  0001 C CNN
-F 4 "DNP" H 10400 3400 50  0001 C CNN "MPN"
-	1    10400 3400
+P 10650 3400
+F 0 "R?" H 10591 3354 50  0000 R CNN
+F 1 "10k" H 10591 3445 50  0000 R CNN
+F 2 "Resistor_SMD:R_0603_1608Metric" H 10650 3400 50  0001 C CNN
+F 3 "~" H 10650 3400 50  0001 C CNN
+F 4 "DNP" H 10650 3400 50  0001 C CNN "MPN"
+	1    10650 3400
 	-1   0    0    1
 $EndComp
 Wire Wire Line
-	10400 3050 10400 3150
+	10650 3050 10650 3150
 Text Label 9900 3250 2    50   ~ 0
 SDA
@@
 Wire Wire Line
 	5900 1750 5950 1750
+Text HLabel 10200 3450 2    50   Output ~ 0
+~INT_PMC
+Wire Wire Line
+	10200 3450 10150 3450
+Connection ~ 10150 3450
+Text HLabel 8250 3450 0    50   Input ~ 0
+EN_SINK
+Wire Wire Line
+	8250 3450 8300 3450
 $EndSCHEMATC

Commit message: Add some part numbers, more changes
Parts:
- removed C?: 1nF, Capacitor_SMD:C_0603_1608Metric, symbol Device:C_Small
- removed D? (x2): 12V, Diode_SMD:D_SOD-523, symbol Device:D_Zener_Small
- removed J?: Jack-DC, Connector_BarrelJack:BarrelJack_Horizontal, symbol Connector:Jack-DC
- removed Q? (x3): 40V, Package_SO:Vishay_PowerPAK_1212-8_Single, symbol Device:Q_NMOS_SGD
- removed R?: 1M, Resistor_SMD:R_0603_1608Metric, symbol Device:R_Small
- removed R?: 100k, Resistor_SMD:R_0603_1608Metric, symbol Device:R_Small
- removed TP?: VBUS_DC, TestPoint:TestPoint_THTPad_D2.0mm_Drill1.0mm, symbol Connector:TestPoint_Small
- removed TP?: ACDRV2, TestPoint:TestPoint_THTPad_D2.0mm_Drill1.0mm, symbol Connector:TestPoint_Small
- C202, C203, C207: renamed from C?; JLC (none) -> 0603; LCSC (none) -> C14663; MPN (none) -> CC0603KRX7R9BB104
- R201, R202, R204, R205, R206: renamed from R?; JLC (none) -> 0603; LCSC (none) -> C25804
- U202: renamed from U?; JLC (none) -> MSOP-10_3.0x3.0x0.5P; LCSC (none) -> C11355; MPN (none) -> FSUSB42MUX
- gave numbers to parts that had none: 14
Connections:
- net labels removed: ACDRV2, VAC2
- wire segments 157 -> 124
Other:
- note removed: "XT60 or spring-loaded\nsockets here?"
- moved on the sheet: C201, C202, C203, C204, C205, C206, C207, D201, D202, J201, Q201, Q202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

Commit message: Schematic is done now
Parts:
- added D201: 5V6, Diode_SMD:D_MiniMELF, symbol Device:D_Zener_Small
- added D202: 3V3, Diode_SMD:D_MiniMELF, symbol Device:D_Zener_Small
- added D204: 5V, Diode_SMD:D_SOD-123, symbol Device:D_Schottky_Small
- added Q202: 40V, Package_TO_SOT_SMD:SOT-23, symbol Device:Q_PMOS_GSD
- added R201: 100, Resistor_SMD:R_1206_3216Metric, symbol Device:R_Small
- added R202: 1k, Resistor_SMD:R_0603_1608Metric, symbol Device:R_Small
- added SW201: Dead Battery, Automated:SW_SPST_PTS636_G, symbol Switch:SW_Push
- C202: renamed from C201; footprint Capacitor_SMD:C_0603_1608Metric -> Capacitor_SMD:C_0402_1005Metric; JLC (none) -> 0402; LCSC (none) -> C1523
- renumbered C203 to C201, C204 to C203, C205 to C204, C206 to C205, C207 to C206, C202 to C207, D201 to D203, D202 to D205, Q202 to Q203, R201 to R204, R202 to R205, R204 to R206, R205 to R207, R206 to R208, U203 to U202, U202 to U203
Connections:
- net VAC1: now also R201.1
- net VBUS: now also D204.1 (K), SW201.2
- new net: D204.2 (A), Q202.3 (D)
- new net: D202.2 (A), Q202.1 (G), R202.2
- new net: D201.1 (K), Q202.2 (S), R201.2
- new net: R202.1, SW201.1
- new net: D201.2 (A), D202.1 (K)
Other:
- note added: "Press to power up the DC/DC \nwhen no battery is attached\nor in case of battery UVLO"
- moved on the sheet: C201, C202, C203, C204, C205, C206, C207, D203, D205, J201, Q201, Q203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

Commit message: Start with layout
Parts:
- C207: footprint Capacitor_SMD:C_0603_1608Metric -> Capacitor_SMD:C_0402_1005Metric; JLC 0603 -> 0402; LCSC C14663 -> (none); MPN CC0603KRX7R9BB104 -> (none)
Changed lines of the file:
@@
 F 0 "C207" V 8921 4650 50  0000 C CNN
 F 1 "100nF" V 9012 4650 50  0000 C CNN
-F 2 "Capacitor_SMD:C_0603_1608Metric" H 9150 4650 50  0001 C CNN
+F 2 "Capacitor_SMD:C_0402_1005Metric" H 9150 4650 50  0001 C CNN
 F 3 "~" H 9150 4650 50  0001 C CNN
-F 4 "0603" H 9150 4650 50  0001 C CNN "JLC"
-F 5 "C14663" H 9150 4650 50  0001 C CNN "LCSC"
-F 6 "CC0603KRX7R9BB104" H 9150 4650 50  0001 C CNN "MPN"
+F 4 "0402" H 9150 4650 50  0001 C CNN "JLC"
+F 5 "" H 9150 4650 50  0001 C CNN "LCSC"
+F 6 "" H 9150 4650 50  0001 C CNN "MPN"
 	1    9150 4650
 	0    1    1    0

Commit message: placed to 50x50mm, started to route
Parts:
- added D206: 3V3, Diode_SMD:D_MiniMELF, symbol Device:D_Zener_Small
- added NT1: UwU, NetTie:NetTie-2_SMD_Pad0.5mm, symbol Device:Net-Tie_2
- D203: value 12V -> 5V6; footprint Diode_SMD:D_SOD-523 -> Diode_SMD:D_MiniMELF; JLC (none) -> LL-34; LCSC (none) -> C8062; MPN (none) -> ZMM5V6
- Q201, Q203: symbol Device:Q_NMOS_SGD -> Transistor_FET:Si7336ADP
- R203, R206: footprint Resistor_SMD:R_0603_1608Metric -> Resistor_SMD:R_0402_1005Metric
Connections:
- net ACDRV1: now also Q201.4 (G), Q203.4 (G); no longer Q201.2 (G), Q203.2 (G)
- net VAC1: now also NT1.1; no longer J201.A4 (VBUS), J201.A9 (VBUS), J201.B4 (VBUS), J201.B9 (VBUS), Q201.3 (D), R201.1
- net VBUS: now also Q203.5 (D); no longer Q203.3 (D)
- net at C202.2, Q201.1 (S), Q203.1 (S): now also Q201.2 (S), Q201.3 (S), Q203.2 (S), Q203.3 (S), D206.2 (A); no longer D203.2 (A)
- new net: D203.2 (A), D206.1 (K)
- new net VBUSRAW: J201.A4 (VBUS), J201.A9 (VBUS), J201.B4 (VBUS), J201.B9 (VBUS), NT1.2, Q201.5 (D), R201.1
Other:
- moved on the sheet: C202, C203, C204, C205, C206, C207, D201, D202, D204, D205, J201, Q201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

Commit message: partially routed
Connections:
- net VBS: now reaches C202.2, D206.2 (A), Q201.1 (S), Q201.2 (S), Q201.3 (S), Q203.1 (S), Q203.2 (S), Q203.3 (S)
Changed lines of the file:
@@
 	0    1    1    0
 $EndComp
+Text Label 4500 2250 0    50   ~ 0
+VBS
 $EndSCHEMATC

Commit message: fully routed but silk is still not done
Changed lines of the file:
@@
 Text Label 9450 2450 2    50   ~ 0
 SCL
-Wire Wire Line
-	9450 2450 9250 2450
-Wire Wire Line
-	9250 2350 9450 2350
 Text Label 9300 2550 0    50   ~ 0
 ~INT_PMC
@@
 Text Label 4500 2250 0    50   ~ 0
 VBS
+Text HLabel 9700 2150 2    50   Input ~ 0
+SCL
+Text HLabel 9700 2050 2    50   BiDi ~ 0
+SDA
+Wire Wire Line
+	9600 2450 9600 2150
+Wire Wire Line
+	9600 2150 9700 2150
+Wire Wire Line
+	9250 2450 9600 2450
+Wire Wire Line
+	9500 2350 9500 2050
+Wire Wire Line
+	9500 2050 9700 2050
+Wire Wire Line
+	9250 2350 9500 2350
 $EndSCHEMATC

Commit message: Add a few more PNs, change D401 to a standard part
Parts:
- C203: JLC (none) -> 0603; LCSC (none) -> C15849; MPN (none) -> CL10A105KB8NNNC
- D205: JLC (none) -> SOD-123; LCSC (none) -> C8598; MPN BAT54W -> B5819W
- R203: JLC (none) -> 0402; LCSC (none) -> C25741
- R206: JLC 0603 -> 0402; LCSC C25804 -> C25744
Changed lines of the file:
@@
 F 1 "1uF" H 5158 6545 50  0000 R CNN
 F 2 "Capacitor_SMD:C_0603_1608Metric" H 5250 6500 50  0001 C CNN
-F 3 "~" H 5250 6500 50  0001 C CNN
+F 3 "https://datasheet.lcsc.com/szlcsc/Samsung-Electro-Mechanics-CL10A105KB8NNNC_C15849.pdf" H 5250 6500 50  0001 C CNN
+F 4 "C15849" H 5250 6500 50  0001 C CNN "LCSC"
+F 5 "0603" H 5250 6500 50  0001 C CNN "JLC"
+F 6 "CL10A105KB8NNNC" H 5250 6500 50  0001 C CNN "MPN"
 	1    5250 6500
 	-1   0    0    1
@@
 F 2 "Resistor_SMD:R_0402_1005Metric" H 5050 6050 50  0001 C CNN
 F 3 "~" H 5050 6050 50  0001 C CNN
+F 4 "0402" V 5050 6050 50  0001 C CNN "JLC"
+F 5 "C25741" V 5050 6050 50  0001 C CNN "LCSC"
 	1    5050 6050
 	0    1    1    0
@@
 F 2 "Diode_SMD:D_SOD-123" V 8150 1550 50  0001 C CNN
 F 3 "~" V 8150 1550 50  0001 C CNN
-F 4 "BAT54W" H 8150 1550 50  0001 C CNN "MPN"
+F 4 "B5819W" H 8150 1550 50  0001 C CNN "MPN"
+F 5 "C8598" H 8150 1550 50  0001 C CNN "LCSC"
+F 6 "SOD-123" H 8150 1550 50  0001 C CNN "JLC"
 	1    8150 1550
 	1    0    0    -1
@@
 F 2 "Resistor_SMD:R_0402_1005Metric" H 9700 2400 50  0001 C CNN
 F 3 "~" H 9700 2400 50  0001 C CNN
-F 4 "0603" H 9700 2400 50  0001 C CNN "JLC"
-F 5 "C25804" H 9700 2400 50  0001 C CNN "LCSC"
+F 4 "0402" H 9700 2400 50  0001 C CNN "JLC"
+F 5 "C25744" H 9700 2400 50  0001 C CNN "LCSC"
 	1    9700 2400
 	-1   0    0    1
