File: input.sch (KiCad schematic (older format))
At the start: 32 parts, among them J201 Power, Q201 40V, Q202 40V, Q203 40V, SW201 Dead Battery, U201 TPD6S300A, U202 FUSB307BMPX, U203 FSUSB42MUX

Commit message: finished routing. no silk artwork.
Parts:
- renumbered D206 to D204, D204 to D205, D205 to D206, NT1 to NT201
Changed lines of the file:
@@
 	8350 1550 8250 1550
 $Comp
-L Device:D_Schottky_Small D205
+L Device:D_Schottky_Small D206
 U 1 1 5F02EFE2
 P 8150 1550
-F 0 "D205" H 8150 1757 50  0000 C CNN
+F 0 "D206" H 8150 1757 50  0000 C CNN
 F 1 "10V" H 8150 1666 50  0000 C CNN
 F 2 "Diode_SMD:D_SOD-123" V 8150 1550 50  0001 C CNN
@@
 P 5000 2850
 AR Path="/5EF44CB5/5F001544" Ref="D?"  Part="1"
-AR Path="/5EFEA158/5F001544" Ref="D204"  Part="1"
-F 0 "D204" H 5000 2643 50  0000 C CNN
+AR Path="/5EFEA158/5F001544" Ref="D205"  Part="1"
+F 0 "D205" H 5000 2643 50  0000 C CNN
 F 1 "5V" H 5000 2734 50  0000 C CNN
 F 2 "Diode_SMD:D_SOD-123" V 5000 2850 50  0001 C CNN
@@
 	3650 3250 3950 3250
 $Comp
-L Device:Net-Tie_2 NT1
+L Device:Net-Tie_2 NT201
 U 1 1 5F0180C7
 P 2950 2000
-F 0 "NT1" H 2950 2089 50  0000 C CNN
+F 0 "NT201" H 2950 2089 50  0000 C CNN
 F 1 "UwU" H 2950 2090 50  0001 C CNN
 F 2 "NetTie:NetTie-2_SMD_Pad0.5mm" H 2950 2000 50  0001 C CNN
@@
 $EndComp
 $Comp
-L Device:D_Zener_Small D206
+L Device:D_Zener_Small D204
 U 1 1 5F3A1EC1
 P 4450 1950
-F 0 "D206" V 4404 2020 50  0000 L CNN
+F 0 "D204" V 4404 2020 50  0000 L CNN
 F 1 "3V3" V 4495 2020 50  0000 L CNN
 F 2 "Diode_SMD:D_MiniMELF" V 4450 1950 50  0001 C CNN

Commit message: Add a few more parts, fix PCB origin problem
Parts:
- C205: JLC (none) -> 0603; LCSC (none) -> C15849
Changed lines of the file:
@@
 F 2 "Capacitor_SMD:C_0603_1608Metric" H 8950 1550 50  0001 C CNN
 F 3 "~" H 8950 1550 50  0001 C CNN
+F 4 "C15849" V 8950 1550 50  0001 C CNN "LCSC"
+F 5 "0603" V 8950 1550 50  0001 C CNN "JLC"
 	1    8950 1550
 	0    -1   -1   0

Commit message: added missing JLC/LCSC parts
Other:
- note added: "2 zeners in series only because\nthis way we can use LCSC basic parts\nand save on the ext. part setup fee"
Changed lines of the file:
@@
 Wire Wire Line
 	9250 2350 9500 2350
+Text Notes 2650 1300 0    50   ~ 0
+2 zeners in series only because\nthis way we can use LCSC basic parts\nand save on the ext. part setup fee
+Wire Notes Line
+	4350 1850 3550 1850
+Wire Notes Line
+	3550 1850 3550 1350
 $EndSCHEMATC

Commit message: updated USB protection IC with package 3D model
Parts:
- U201: footprint Package_DFN_QFN:QFN-20-1EP_3x3mm_P0.4mm_EP1.65x1.65mm -> Automated:QFN-20-1EP_3x3mm_P0.4mm_EP1.65x1.65mm
Changed lines of the file:
@@
 F 0 "U201" H 3550 6515 50  0000 C CNN
 F 1 "TPD6S300A" H 3550 6424 50  0000 C CNN
-F 2 "Package_DFN_QFN:QFN-20-1EP_3x3mm_P0.4mm_EP1.65x1.65mm" H 3700 5850 50  0001 C CNN
+F 2 "Automated:QFN-20-1EP_3x3mm_P0.4mm_EP1.65x1.65mm" H 3700 5850 50  0001 C CNN
 F 3 "https://www.ti.com/lit/ds/symlink/tpd6s300a.pdf" H 3550 5950 50  0001 C CNN
 F 4 "TPD6S300ARUKR" H 3550 5923 50  0001 C CNN "MPN"

Commit message: added 3D models
Parts:
- J201: footprint Connector_USB:USB_C_Receptacle_XKB_U262-16XN-4BVC11 -> Automated:USB_C_Receptacle_XKB_U262-16XN-4BVC11
- Q201, Q203: footprint Package_SO:Vishay_PowerPAK_1212-8_Single -> Automated:Vishay_PowerPAK_1212-8_Single
Changed lines of the file:
@@
 F 0 "J201" H 1821 2789 50  0000 R CNN
 F 1 "Power" H 1821 2698 50  0000 R CNN
-F 2 "Connector_USB:USB_C_Receptacle_XKB_U262-16XN-4BVC11" H 2400 2850 50  0001 C CNN
+F 2 "Automated:USB_C_Receptacle_XKB_U262-16XN-4BVC11" H 2400 2850 50  0001 C CNN
 F 3 "https://www.usb.org/sites/default/files/documents/usb_type-c.zip" H 2400 2850 50  0001 C CNN
 	1    2250 2850
@@
 F 0 "Q201" V 4349 2150 50  0000 C CNN
 F 1 "40V" V 4440 2150 50  0000 C CNN
-F 2 "Package_SO:Vishay_PowerPAK_1212-8_Single" H 4300 2250 50  0001 C CNN
+F 2 "Automated:Vishay_PowerPAK_1212-8_Single" H 4300 2250 50  0001 C CNN
 F 3 "~" H 4100 2150 50  0001 C CNN
 F 4 "SiSS10ADN" V 4100 2150 50  0001 C CNN "MPN"
@@
 F 0 "Q203" V 5349 2150 50  0000 C CNN
 F 1 "40V" V 5440 2150 50  0000 C CNN
-F 2 "Package_SO:Vishay_PowerPAK_1212-8_Single" H 5300 2250 50  0001 C CNN
+F 2 "Automated:Vishay_PowerPAK_1212-8_Single" H 5300 2250 50  0001 C CNN
 F 3 "~" H 5100 2150 50  0001 C CNN
 F 4 "SiSS10ADN" V 5100 2150 50  0001 C CNN "MPN"
