File: control.sch (KiCad schematic (older format))
At the start: 46 parts, among them J10 CTRL, J11 RS485, J12 CHG, J13 SOICbite, SW1 RESET, SW2 USER, U6 STM32F072CBTx

Commit message: I'm pretty happy with it now, will place tomorrow
Connections:
- net USB_SEL: now reaches U6.38 (PA15)
- no-connect marks 21 -> 20
Changed lines of the file:
@@
 Text Label 2150 1200 0    50   ~ 0
 ~RST
-Text Label 4100 3500 2    50   ~ 0
-D+
-Text Label 4100 3400 2    50   ~ 0
-D-
 NoConn ~ 2450 1600
 NoConn ~ 2450 1700
 NoConn ~ 2450 2000
-NoConn ~ 2450 2100
 Text Label 2100 3100 0    50   ~ 0
 SCL
@@
 	2150 1400 2450 1400
 Wire Wire Line
-	4100 3400 3750 3400
-Wire Wire Line
-	3750 3500 4100 3500
-Text HLabel 2400 2600 0    50   Input ~ 0
+	3850 3400 3750 3400
+Wire Wire Line
+	3750 3500 3850 3500
+Text HLabel 2350 2600 0    50   Input ~ 0
 ~INT_PMC
-Text HLabel 2400 2500 0    50   Input ~ 0
+Text HLabel 2350 2500 0    50   Input ~ 0
 ~INT_CHG
-Text HLabel 2400 2400 0    50   Input ~ 0
+Text HLabel 2350 2400 0    50   Input ~ 0
 EN_SNK
-Text HLabel 2400 2300 0    50   Output ~ 0
+Text HLabel 2350 2300 0    50   Output ~ 0
 ~CE
 Text HLabel 4450 1200 0    50   Output ~ 0
@@
 SDA
 Wire Wire Line
-	2450 2600 2400 2600
-Wire Wire Line
-	2400 2500 2450 2500
-Wire Wire Line
-	2450 2400 2400 2400
-Wire Wire Line
-	2400 2300 2450 2300
+	2450 2600 2350 2600
+Wire Wire Line
+	2350 2500 2450 2500
+Wire Wire Line
+	2450 2400 2350 2400
+Wire Wire Line
+	2350 2300 2450 2300
 Text Label 2100 2900 0    50   ~ 0
 UART_TX
@@
 Wire Wire Line
 	8250 4900 8250 5000
-NoConn ~ 3750 3800
 Text Notes 1650 850  0    50   ~ 0
 TODO: BOOT0 selector switch
@@
 Wire Wire Line
 	5700 5850 6250 5850
-Text Label 4400 3200 2    50   ~ 0
+Text Label 4350 3200 2    50   ~ 0
 USB_UART_TX
 Wire Wire Line
-	4400 3200 3750 3200
-Text Label 4400 3300 2    50   ~ 0
+	4350 3200 3750 3200
+Text Label 4350 3300 2    50   ~ 0
 USB_UART_RX
 Wire Wire Line
-	4400 3300 3750 3300
-Text Label 2100 3300 0    50   ~ 0
-SBU2
-Text Label 2100 3400 0    50   ~ 0
-SBU1
-Wire Wire Line
-	2450 3400 2100 3400
-Wire Wire Line
-	2100 3300 2450 3300
+	4350 3300 3750 3300
 Wire Wire Line
 	8650 2600 8650 2850
@@
 Text Label 8950 2850 1    50   ~ 0
 Blue2
-Text Label 4050 2300 2    50   ~ 0
-SBU1
-Text Label 4050 2400 2    50   ~ 0
-SBU2
-Wire Wire Line
-	3750 2400 4050 2400
-Wire Wire Line
-	4050 2300 3750 2300
 Text Label 2100 3600 0    50   ~ 0
 EXT_SCL
@@
 NoConn ~ 3750 2800
 NoConn ~ 3750 3100
+Text HLabel 3850 3400 2    50   BiDi ~ 0
+D-
+Text HLabel 3850 3500 2    50   BiDi ~ 0
+D+
+Text HLabel 3850 2300 2    50   BiDi ~ 0
+SBU1
+Text HLabel 2350 3400 0    50   BiDi ~ 0
+SBU1
+Wire Wire Line
+	2450 3300 2350 3300
+Wire Wire Line
+	3850 2300 3750 2300
+Text HLabel 3850 2400 2    50   BiDi ~ 0
+SBU2
+Wire Wire Line
+	3850 2400 3750 2400
+Text HLabel 2350 3300 0    50   BiDi ~ 0
+SBU2
+Wire Wire Line
+	2450 3400 2350 3400
+NoConn ~ 2450 2100
+Text HLabel 3850 3800 2    50   Output ~ 0
+USB_SEL
+Wire Wire Line
+	3850 3800 3750 3800
 $EndSCHEMATC

Commit message: Add some part numbers, more changes
Parts:
- removed C30, C34, C35: 100nF, Capacitor_SMD:C_0603_1608Metric, symbol Device:C_Small
- removed C36: 1uF, Capacitor_SMD:C_0603_1608Metric, symbol Device:C_Small
- removed C?: 10nF, Capacitor_SMD:C_0402_1005Metric, symbol Device:C_Small
- removed C?: 100nF, Capacitor_SMD:C_0402_1005Metric, symbol Device:C_Small
- removed D8: D_TVS, symbol Device:D_TVS
- added C403: 10nF, Capacitor_SMD:C_0402_1005Metric, symbol Device:C_Small
- added C404, C408, C409, C410: 100nF, Capacitor_SMD:C_0402_1005Metric, symbol Device:C_Small
- added C411: 1uF, Capacitor_SMD:C_0402_1005Metric, symbol Device:C_Small
- added D403: 5V, Diode_SMD:D_SOD-523, symbol Device:D_TVS
- added R402: 10k, Resistor_SMD:R_0603_1608Metric, symbol Device:R_Small
- C405: renamed from C31; footprint Capacitor_SMD:C_0603_1608Metric -> Capacitor_SMD:C_0402_1005Metric; JLC (none) -> 0402; LCSC (none) -> C52923
- C406: renamed from C32; footprint Capacitor_SMD:C_0603_1608Metric -> Capacitor_SMD:C_0402_1005Metric; JLC (none) -> 0402; LCSC (none) -> C1525; MPN (none) -> CL05B104KO5NNNC
- C407: renamed from C33; JLC (none) -> 0603; LCSC (none) -> C19666; MPN (none) -> CL10A475KO8NNNC
- C412: renamed from C37; footprint Capacitor_SMD:C_0603_1608Metric -> Capacitor_SMD:C_0402_1005Metric; JLC (none) -> 0402; LCSC (none) -> C15195
- D404: renamed from D9; value D_TVS -> 5V; footprint (none) -> Diode_SMD:D_SOD-523
- R401: renamed from R19; JLC (none) -> 0603; LCSC (none) -> C25804
- R403: renamed from R20; JLC (none) -> 0603; LCSC (none) -> C25804
- R406: renamed from R21; JLC (none) -> 0603; LCSC (none) -> C22775; MPN (none) -> 0603WAF1000T5E
- R407: renamed from R22; JLC (none) -> 0603; LCSC (none) -> C22775; MPN (none) -> 0603WAF1000T5E
- R408: renamed from R23; JLC (none) -> 0603; LCSC (none) -> C22775; MPN (none) -> 0603WAF1000T5E
- R409: renamed from R24; JLC (none) -> 0603; LCSC (none) -> C22775; MPN (none) -> 0603WAF1000T5E
- R410: renamed from R25; JLC (none) -> 0603; LCSC (none) -> C22775; MPN (none) -> 0603WAF1000T5E
- R411: renamed from R16; JLC (none) -> 0603; LCSC (none) -> C22775; MPN (none) -> 0603WAF1000T5E
- R412: renamed from R17; JLC (none) -> 0603; LCSC (none) -> C25804
- R413: renamed from R18; JLC (none) -> 0603; LCSC (none) -> C25804
- U401: renamed from U6; JLC (none) -> LQFP-48_7.0x7.0x0.5P; LCSC (none) -> C80488; MPN (none) -> STM32F072C8T6
- U402: renamed from U?; JLC (none) -> SOIC-16_3.9x9.9x1.27P; LCSC (none) -> C14267; MPN (none) -> CH340G
- U403: renamed from U?; JLC (none) -> SOIC-8_3.9x4.9x1.27P; LCSC (none) -> C8963; MPN (none) -> SP3485EN-L/TR
- gave numbers to parts that had none: 3
- renumbered D6 to D401, D7 to D402, D10 to D405, D11 to D406, D12 to D407, D13 to D408, D14 to D409, D15 to D410, J12 to J401, J10 to J402, J13 to J403, J11 to J404, R26 to R404, R27 to R405, SW1 to SW401, SW2 to SW402, TP7 to TP401, TP8 to TP402
Connections:
- net +3V3: now also C404.2, C408.1, C409.1, C410.2, C411.1
- net BOOT0: now also R402.1
- net D+: now also D403.1 (A1)
- net GND: now also C403.2, C404.1, C408.2, C409.2, C410.1, C411.2, D403.2 (A2), R402.2
- net at U402.4 (V3): now also C403.1
Other:
- moved on the sheet: R401, SW401

Commit message: Schematic is done now
Parts:
- D401: footprint (none) -> Diode_SMD:D_SOD-323; JLC (none) -> SOD-323; LCSC (none) -> C116441; MPN (none) -> MM3Z27VT1G
- D402: value TODO -> 30V; JLC (none) -> SOD-123; LCSC (none) -> C8598; MPN (none) -> B5819W
- J403: footprint (none) -> ferret:SOIC_clipProgSmall
- renumbered D410 to D406, D406 to D407, D407 to D408, D408 to D409, D409 to D410
Connections:
- net GND: now also J403.4 (Pin_4); no longer J403.1 (Pin_1), J403.5 (Pin_5)
- net SWCLK: now also J403.7 (Pin_7); no longer J403.6 (Pin_6)
- net SWDIO: now also J403.5 (Pin_5); no longer J403.7 (Pin_7)
- net ~RST: now also J403.8 (Pin_8); no longer J403.3 (Pin_3)
- removed net SOIC_3V3: D406.2 (A), J403.4 (Pin_4), J403.8 (Pin_8)
- new net: D406.2 (A), J403.1 (Pin_1)
- no-connect marks 20 -> 22
Other:
- moved on the sheet: C401, C402, D406, Y401

Commit message: Start with layout
Parts:
- added NT401: VDDA, NetTie:NetTie-2_SMD_Pad0.5mm, symbol Device:Net-Tie_2
- added NT402: VDDIO2, NetTie:NetTie-2_SMD_Pad0.5mm, symbol Device:Net-Tie_2
- added NT403: VDD, NetTie:NetTie-2_SMD_Pad0.5mm, symbol Device:Net-Tie_2
Connections:
- net +3V3: now also NT401.1, NT402.1, NT403.1; no longer C405.1, C406.1, C407.1, C408.1, C409.1, C411.1, C412.1, U401.1 (VBAT), U401.24 (VDD), U401.36 (VDDIO2), U401.48 (VDD), U401.9 (VDDA)
- new net VDD: C407.1, C408.1, C409.1, NT403.2, U401.1 (VBAT), U401.24 (VDD), U401.48 (VDD)
- new net VDDA: C411.1, C412.1, NT401.2, U401.9 (VDDA)
- new net VDDIO2: C405.1, C406.1, NT402.2, U401.36 (VDDIO2)
Changed lines of the file:
@@
 L power:+3V3 #PWR0417
 U 1 1 5EF81766
-P 6300 850
-F 0 "#PWR0417" H 6300 700 50  0001 C CNN
-F 1 "+3V3" H 6315 1023 50  0000 C CNN
-F 2 "" H 6300 850 50  0001 C CNN
-F 3 "" H 6300 850 50  0001 C CNN
-	1    6300 850
+P 6300 550
+F 0 "#PWR0417" H 6300 400 50  0001 C CNN
+F 1 "+3V3" H 6315 723 50  0000 C CNN
+F 2 "" H 6300 550 50  0001 C CNN
+F 3 "" H 6300 550 50  0001 C CNN
+	1    6300 550
 	1    0    0    -1
 $EndComp
@@
 $EndComp
 Wire Wire Line
-	6300 850  6300 900
+	6300 550  6300 600
 Text Label 5600 900  0    50   ~ 0
 VDDIO2
@@
 L power:+3V3 #PWR0419
 U 1 1 5EF8E890
-P 7800 850
-F 0 "#PWR0419" H 7800 700 50  0001 C CNN
-F 1 "+3V3" H 7815 1023 50  0000 C CNN
-F 2 "" H 7800 850 50  0001 C CNN
-F 3 "" H 7800 850 50  0001 C CNN
-	1    7800 850
+P 7800 550
+F 0 "#PWR0419" H 7800 400 50  0001 C CNN
+F 1 "+3V3" H 7815 723 50  0000 C CNN
+F 2 "" H 7800 550 50  0001 C CNN
+F 3 "" H 7800 550 50  0001 C CNN
+	1    7800 550
 	1    0    0    -1
 $EndComp
@@
 Connection ~ 7400 900
 Wire Wire Line
-	7800 900  7800 850
+	7800 900  7800 800
 Connection ~ 7800 900
 Wire Wire Line
@@
 L power:+3V3 #PWR0426
 U 1 1 5EF935B7
-P 8950 850
-F 0 "#PWR0426" H 8950 700 50  0001 C CNN
-F 1 "+3V3" H 8965 1023 50  0000 C CNN
-F 2 "" H 8950 850 50  0001 C CNN
-F 3 "" H 8950 850 50  0001 C CNN
-	1    8950 850
+P 8950 550
+F 0 "#PWR0426" H 8950 400 50  0001 C CNN
+F 1 "+3V3" H 8965 723 50  0000 C CNN
+F 2 "" H 8950 550 50  0001 C CNN
+F 3 "" H 8950 550 50  0001 C CNN
+	1    8950 550
 	1    0    0    -1
 $EndComp
@@
 $EndComp
 Wire Wire Line
-	8950 850  8950 900
+	8950 550  8950 600
 Text Label 8250 900  0    50   ~ 0
 VDDA
@@
 NoConn ~ 8100 3950
 NoConn ~ 8600 3950
+$Comp
+L Device:Net-Tie_2 NT401
+U 1 1 5F08D247
+P 8950 700
+F 0 "NT401" V 8950 744 50  0000 L CNN
+F 1 "VDDA" V 8995 744 50  0001 L CNN
+F 2 "NetTie:NetTie-2_SMD_Pad0.5mm" H 8950 700 50  0001 C CNN
+F 3 "~" H 8950 700 50  0001 C CNN
+F 4 "DNP" V 8950 700 50  0001 C CNN "MPN"
+	1    8950 700
+	0    1    1    0
+$EndComp
+Wire Wire Line
+	8950 800  8950 900
+$Comp
+L Device:Net-Tie_2 NT403
+U 1 1 5F0ACE23
+P 7800 700
+F 0 "NT403" V 7800 744 50  0000 L CNN
+F 1 "VDD" V 7845 744 50  0001 L CNN
+F 2 "NetTie:NetTie-2_SMD_Pad0.5mm" H 7800 700 50  0001 C CNN
+F 3 "~" H 7800 700 50  0001 C CNN
+F 4 "DNP" V 7800 700 50  0001 C CNN "MPN"
+	1    7800 700
+	0    1    1    0
+$EndComp
+Wire Wire Line
+	7800 600  7800 550
+$Comp
+L Device:Net-Tie_2 NT402
+U 1 1 5F0B99EA
+P 6300 700
+F 0 "NT402" V 6300 744 50  0000 L CNN
+F 1 "VDDIO2" V 6345 744 50  0001 L CNN
+F 2 "NetTie:NetTie-2_SMD_Pad0.5mm" H 6300 700 50  0001 C CNN
+F 3 "~" H 6300 700 50  0001 C CNN
+F 4 "DNP" V 6300 700 50  0001 C CNN "MPN"
+	1    6300 700
+	0    1    1    0
+$EndComp
+Wire Wire Line
+	6300 800  6300 900
 $EndSCHEMATC

Commit message: placed to 50x50mm, started to route
Parts:
- removed R406, R407, R408, R409: 100, Resistor_SMD:R_0603_1608Metric, symbol Device:R_Small
- added R406: 470, Resistor_SMD:R_Array_Convex_4x0603, symbol Device:R_Pack04
- Y401: symbol Device:Crystal_Small -> Device:Crystal_GND24_Small
Connections:
- net +3V3: now also R406.5 (R4.2), R406.6 (R3.2), R406.7 (R2.2), R406.8 (R1.2)
- net GND: now also Y401.2, Y401.4
- net at D409.2 (A): now also R406.1 (R1.1)
- net at D405.2 (A): now also R406.4 (R4.1)
- net at D407.2 (A): now also R406.3 (R3.1)
- net at D408.2 (A): now also R406.2 (R2.1)
- net XT_N: now reaches C402.1, U402.8 (XO)
- net XT_N: now also Y401.3; no longer Y401.2
- net XT_P: now reaches C401.1, U402.7 (XI), Y401.1
- net A renamed RS485_P
- net B renamed RS485_N
Other:
- moved on the sheet: C401, C402, C403, C404, C405, C406, C407, C408, C409, C410, C411, C412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

Commit message: partially routed
Parts:
- R410: value 100 -> 470; LCSC C22775 -> (none); MPN 0603WAF1000T5E -> (none)
Connections:
- net D+: no longer D403.1 (A1), J402.A6 (D+), J402.B6 (D+), U402.5 (UD+)
- net D-: no longer D404.1 (A1), J402.A7 (D-), J402.B7 (D-), U402.6 (UD-)
- new net SCD+: D403.1 (A1), J402.A6 (D+), J402.B6 (D+), U402.5 (UD+)
- new net SCD-: D404.1 (A1), J402.A7 (D-), J402.B7 (D-), U402.6 (UD-)
Other:
- moved on the sheet: D403
Changed lines of the file:
@@
 P 9200 2750
 F 0 "R410" H 9141 2796 50  0000 R CNN
-F 1 "100" H 9141 2705 50  0000 R CNN
+F 1 "470" H 9141 2705 50  0000 R CNN
 F 2 "Resistor_SMD:R_0603_1608Metric" H 9200 2750 50  0001 C CNN
 F 3 "https://datasheet.lcsc.com/szlcsc/Uniroyal-Elec-0603WAF1000T5E_C22775.pdf" H 9200 2750 50  0001 C CNN
 F 4 "0603" H 9200 2750 50  0001 C CNN "JLC"
-F 5 "C22775" H 9200 2750 50  0001 C CNN "LCSC"
-F 6 "0603WAF1000T5E" H 9200 2750 50  0001 C CNN "MPN"
+F 5 "" H 9200 2750 50  0001 C CNN "LCSC"
+F 6 "" H 9200 2750 50  0001 C CNN "MPN"
 	1    9200 2750
 	-1   0    0    -1
@@
 	3300 6300 2550 6300
 Wire Wire Line
-	2950 6500 2950 6550
-Wire Wire Line
-	2950 6500 2550 6500
-Wire Wire Line
-	2950 6500 3150 6500
-Connection ~ 2950 6500
+	2900 6500 2900 6550
+Wire Wire Line
+	2900 6500 2550 6500
+Wire Wire Line
+	2900 6500 3150 6500
+Connection ~ 2900 6500
 Text Label 3150 6500 2    50   ~ 0
-D+
-Wire Wire Line
-	3300 6300 3500 6300
+SCD+
+Wire Wire Line
+	3300 6300 3550 6300
 Connection ~ 3300 6300
-Text Label 3500 6300 2    50   ~ 0
-D-
+Text Label 3550 6300 2    50   ~ 0
+SCD-
 $Comp
 L power:GND #PWR0408
@@
 L power:GND #PWR0406
 U 1 1 5EF3BF88
-P 2950 6900
-F 0 "#PWR0406" H 2950 6650 50  0001 C CNN
-F 1 "GND" H 2872 6863 50  0000 R CNN
-F 2 "" H 2950 6900 50  0001 C CNN
-F 3 "" H 2950 6900 50  0001 C CNN
-	1    2950 6900
-	-1   0    0    -1
-$EndComp
-Wire Wire Line
-	2950 6900 2950 6850
+P 2900 6900
+F 0 "#PWR0406" H 2900 6650 50  0001 C CNN
+F 1 "GND" H 2822 6863 50  0000 R CNN
+F 2 "" H 2900 6900 50  0001 C CNN
+F 3 "" H 2900 6900 50  0001 C CNN
+	1    2900 6900
+	-1   0    0    -1
+$EndComp
+Wire Wire Line
+	2900 6900 2900 6850
 Wire Wire Line
 	3300 6700 3300 6650
@@
 	-1   0    0    -1
 $EndComp
-Text Label 4900 6500 0    50   ~ 0
-D-
-Text Label 4900 6400 0    50   ~ 0
-D+
-Wire Wire Line
-	4900 6500 5050 6500
-Wire Wire Line
-	5050 6400 4900 6400
+Text Label 4800 6500 0    50   ~ 0
+SCD-
+Text Label 4800 6400 0    50   ~ 0
+SCD+
+Wire Wire Line
+	4800 6500 5050 6500
+Wire Wire Line
+	5050 6400 4800 6400
 NoConn ~ 5050 6200
 Wire Wire Line
@@
 L Device:D_TVS D403
 U 1 1 5EFE80D7
-P 2950 6700
-F 0 "D403" V 2904 6621 50  0000 R CNN
-F 1 "5V" V 2995 6621 50  0000 R CNN
-F 2 "Diode_SMD:D_SOD-523" H 2950 6700 50  0001 C CNN
-F 3 "~" H 2950 6700 50  0001 C CNN
-	1    2950 6700
+P 2900 6700
+F 0 "D403" V 2854 6621 50  0000 R CNN
+F 1 "5V" V 2945 6621 50  0000 R CNN
+F 2 "Diode_SMD:D_SOD-523" H 2900 6700 50  0001 C CNN
+F 3 "~" H 2900 6700 50  0001 C CNN
+	1    2900 6700
 	0    -1   1    0
 $EndComp

Commit message: Add a few more PNs, change D401 to a standard part
Parts:
- removed D401: 20V, Diode_SMD:D_SOD-323, symbol Device:D_Zener_Small
- added D401: 20V, Diode_SMD:D_SOD-123, symbol Device:D_Schottky_Small
- R404, R405: JLC (none) -> 0603; LCSC (none) -> C23162
- R410: LCSC (none) -> C23179
Connections:
- net GND: now also D401.2 (A)
- net at D402.2 (A), J402.A4 (VBUS), J402.A9 (VBUS)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: now also D401.1 (K)
Changed lines of the file:
@@
 F 2 "Resistor_SMD:R_0603_1608Metric" H 5100 1650 50  0001 C CNN
 F 3 "~" H 5100 1650 50  0001 C CNN
+F 4 "0603" H 5100 1650 50  0001 C CNN "JLC"
+F 5 "C23162" H 5100 1650 50  0001 C CNN "LCSC"
 	1    5100 1650
 	-1   0    0    -1
@@
 F 2 "Resistor_SMD:R_0603_1608Metric" H 5200 1650 50  0001 C CNN
 F 3 "~" H 5200 1650 50  0001 C CNN
+F 4 "0603" H 5200 1650 50  0001 C CNN "JLC"
+F 5 "C23162" H 5200 1650 50  0001 C CNN "LCSC"
 	1    5200 1650
 	-1   0    0    -1
@@
 F 3 "https://datasheet.lcsc.com/szlcsc/Uniroyal-Elec-0603WAF1000T5E_C22775.pdf" H 9200 2750 50  0001 C CNN
 F 4 "0603" H 9200 2750 50  0001 C CNN "JLC"
-F 5 "" H 9200 2750 50  0001 C CNN "LCSC"
+F 5 "C23179" H 9200 2750 50  0001 C CNN "LCSC"
 F 6 "" H 9200 2750 50  0001 C CNN "MPN"
 	1    9200 2750
@@
 Wire Wire Line
 	2750 5750 2600 5750
-$Comp
-L Device:D_Zener_Small D401
-U 1 1 5F153A66
-P 2600 5900
-F 0 "D401" V 2554 5830 50  0000 R CNN
-F 1 "20V" V 2645 5830 50  0000 R CNN
-F 2 "Diode_SMD:D_SOD-323" V 2600 5900 50  0001 C CNN
-F 3 "~" V 2600 5900 50  0001 C CNN
-F 4 "MM3Z27VT1G" V 2600 5900 50  0001 C CNN "MPN"
-F 5 "SOD-323" V 2600 5900 50  0001 C CNN "JLC"
-F 6 "C116441" V 2600 5900 50  0001 C CNN "LCSC"
-	1    2600 5900
-	0    -1   1    0
-$EndComp
 Wire Wire Line
 	2600 5800 2600 5750
@@
 Wire Wire Line
 	8900 2950 8900 3200
+$Comp
+L Device:D_Schottky_Small D?
+U 1 1 5F1019A5
+P 2600 5900
+AR Path="/5EFEA158/5F1019A5" Ref="D?"  Part="1"
+AR Path="/5EF44CB5/5F1019A5" Ref="D401"  Part="1"
+F 0 "D401" H 2600 6107 50  0000 C CNN
+F 1 "20V" H 2600 6016 50  0000 C CNN
+F 2 "Diode_SMD:D_SOD-123" V 2600 5900 50  0001 C CNN
+F 3 "~" V 2600 5900 50  0001 C CNN
+F 4 "B5819W" H 2600 5900 50  0001 C CNN "MPN"
+F 5 "C8598" H 2600 5900 50  0001 C CNN "LCSC"
+F 6 "SOD-123" H 2600 5900 50  0001 C CNN "JLC"
+	1    2600 5900
+	0    1    1    0
+$EndComp
 $EndSCHEMATC
