File: ferret.kicad_pcb (KiCad board)
At the start: 4 copper layers, 50 x 50 mm, 135 parts, among them J201 Power, J301 BAT, J302 BAT, J304 SYS, J401 CTRL, J402 CHG, J403 SOICbite, J404 RS485, Q201 40V, Q202 40V, Q203 40V, SW201 Dead Battery, SW401 USER, SW402 RESET, U201 TPD6S300A, U202 FUSB307BMPX, U203 FSUSB42MUX, U301 TPS560430X3F, U302 BQ25792, U401 STM32F072CBTx, U402 CH340G, U403 SP3485EN, Y401 12MHz, Y402 12MHz

Commit message: Add a few more parts, fix PCB origin problem
Changed lines of the file:
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@@
   (general
     (thickness 1.6)
-    (drawings 14)
-    (tracks 1985)
+    (drawings 18)
+    (tracks 1987)
     (zones 0)
     (modules 135)
@@
   (page A4)
   (layers
-    (0 F.Cu signal hide)
+    (0 F.Cu signal)
     (1 In1.Cu power hide)
     (2 In2.Cu mixed hide)
-    (31 B.Cu signal hide)
+    (31 B.Cu signal)
     (32 B.Adhes user hide)
     (33 F.Adhes user hide)
@@
     (36 B.SilkS user)
     (37 F.SilkS user hide)
-    (38 B.Mask user hide)
+    (38 B.Mask user)
     (39 F.Mask user hide)
     (40 Dwgs.User user hide)
@@
   )
   (setup
-    (last_trace_width 0.2)
+    (last_trace_width 0.3)
     (user_trace_width 0.1524)
     (user_trace_width 0.16)
@@
     )
   )
+  (gr_circle (center 129.9 117.4) (end 129.98 117.4) (layer B.SilkS) (width 0.16))
+  (gr_circle (center 146 94.4) (end 146.08 94.4) (layer B.SilkS) (width 0.16))
+  (gr_circle (center 156.7 101.95) (end 156.78 101.95) (layer B.SilkS) (width 0.16))
+  (gr_circle (center 153.15 106.95) (end 153.23 106.95) (layer B.SilkS) (width 0.16))
   (gr_text CTRL (at 169.9 110.2) (layer F.SilkS)
     (effects (font (size 1 1) (thickness 0.15)))
@@
   (segment (start 170.228553 124.353553) (end 172.146447 124.353553) (width 0.2) (layer B.Cu) (net 69))
   (segment (start 153.3 131.4) (end 153.7 131.8) (width 0.3) (layer F.Cu) (net 69))
-  (segment (start 152.7 131.4) (end 153.3 131.4) (width 0.3) (layer F.Cu) (net 69))
   (segment (start 153.8 132.4) (end 154.3 132.9) (width 0.3) (layer F.Cu) (net 69))
   (segment (start 153.8 131.9) (end 153.8 132.4) (width 0.3) (layer F.Cu) (net 69))
@@
   (segment (start 168.1 134.2) (end 170.2 132.1) (width 2) (layer B.Cu) (net 69))
   (segment (start 166.6 134.2) (end 168.1 134.2) (width 2) (layer B.Cu) (net 69))
+  (segment (start 152.7 131.4) (end 153.3 131.4) (width 0.3) (layer F.Cu) (net 69))
   (via (at 140.45 110.975) (size 0.52) (drill 0.26) (layers F.Cu B.Cu) (net 70))
   (via (at 140.55 112.225) (size 0.52) (drill 0.26) (layers F.Cu B.Cu) (net 70))
@@
   (segment (start 151.939305 129.860695) (end 152.839931 128.960069) (width 0.2) (layer B.Cu) (net 78))
   (segment (start 151.702406 129.860695) (end 151.939305 129.860695) (width 0.2) (layer B.Cu) (net 78))
-  (segment (start 154.325 129.275) (end 157.225 129.275) (width 0.4) (layer F.Cu) (net 78))
-  (segment (start 153.625 129.975) (end 154.325 129.275) (width 0.3) (layer F.Cu) (net 78))
-  (segment (start 153.55 130.05) (end 153.625 129.975) (width 0.3) (layer F.Cu) (net 78))
-  (segment (start 152.7 130.05) (end 153.55 130.05) (width 0.3) (layer F.Cu) (net 78))
   (segment (start 163.8 128.2) (end 163.8 124.95) (width 1.4) (layer F.Cu) (net 78))
   (segment (start 162.9 129.1) (end 163.8 128.2) (width 1.4) (layer F.Cu) (net 78))
   (segment (start 162.9 129.1) (end 157.45 129.1) (width 0.8) (layer F.Cu) (net 78))
+  (segment (start 154.325 129.275) (end 154.725 129.275) (width 0.3) (layer F.Cu) (net 78))
+  (segment (start 153.55 130.05) (end 154.325 129.275) (width 0.3) (layer F.Cu) (net 78))
+  (segment (start 152.7 130.05) (end 153.55 130.05) (width 0.3) (layer F.Cu) (net 78))
+  (segment (start 154.725 129.275) (end 157.3 129.275) (width 0.39) (layer F.Cu) (net 78))
+  (segment (start 154.4 129.275) (end 154.725 129.275) (width 0.39) (layer F.Cu) (net 78))
   (via (at 165 135.8) (size 0.5) (drill 0.2) (layers F.Cu B.Cu) (net 79))
   (via (at 165.8 135.8) (size 0.5) (drill 0.2) (layers F.Cu B.Cu) (net 79))
@@
   (segment (start 153.5 130.95) (end 153.575 131.025) (width 0.3) (layer F.Cu) (net 79))
   (segment (start 153.575 131.025) (end 154.375 131.825) (width 0.3) (layer F.Cu) (net 79))
-  (segment (start 154.375 131.825) (end 154.375 131.925) (width 0.2) (layer F.Cu) (net 79))
-  (segment (start 154.375 131.925) (end 157.275 131.925) (width 0.38) (layer F.Cu) (net 79))
+  (segment (start 154.5 131.925) (end 157.4 131.925) (width 0.38) (layer F.Cu) (net 79))
   (segment (start 152.5875 133.479477) (end 152.969989 133.096988) (width 0.2) (layer F.Cu) (net 79))
   (via (at 152.969989 133.096988) (size 0.52) (drill 0.26) (layers F.Cu B.Cu) (net 79))
@@
   (segment (start 163.8 135.8) (end 163.8 136.05) (width 0.8) (layer F.Cu) (net 79))
   (via (at 163.8 135.8) (size 0.5) (drill 0.2) (layers F.Cu B.Cu) (net 79))
+  (segment (start 154.925 131.925) (end 154.96499 131.96499) (width 0.3) (layer F.Cu) (net 79))
+  (segment (start 154.5 131.925) (end 154.925 131.925) (width 0.3) (layer F.Cu) (net 79))
   (segment (start 149.590986 133.4) (end 148.869959 133.4) (width 0.16) (layer F.Cu) (net 80))
   (segment (start 150.2 132.3625) (end 150.2 132.790986) (width 0.16) (layer F.Cu) (net 80))
